Commit message: [Implementation] Added foot frames as end effector frames and computed ground reaction forces. However adjustments are needed.

File: assets/models/go2/go2.urdf (robot description, URDF)
Before this commit: robot go2, 13 links, 12 joints
Links:
- added link FL_ee, mass 0.001; collision sphere radius=0.01
- added link FR_ee, mass 0.001; collision sphere radius=0.01
- added link RL_ee, mass 0.001; collision sphere radius=0.01
- added link RR_ee, mass 0.001; collision sphere radius=0.01
Joints:
- added joint FL_ee_joint: type fixed, parent FL_calf, child FL_ee, origin xyz=0 0 -0.1 rpy=0 0 0
- added joint FR_ee_joint: type fixed, parent FR_calf, child FR_ee, origin xyz=0 0 -0.1 rpy=0 0 0
- added joint RL_ee_joint: type fixed, parent RL_calf, child RL_ee, origin xyz=0 0 -0.1 rpy=0 0 0
- added joint RR_ee_joint: type fixed, parent RR_calf, child RR_ee, origin xyz=0 0 -0.1 rpy=0 0 0

Commit message: [Implementation] Fixed and verified the contact forces computation using rnea.

File: assets/models/go2/go2.urdf (robot description, URDF)
Before this commit: robot go2, 17 links, 16 joints
Links:
- removed link FL_ee
- removed link FR_ee
- removed link RL_ee
- removed link RR_ee
- added link FL_EE, mass 0.001; collision sphere radius=0.01
- added link FR_EE, mass 0.001; collision sphere radius=0.01
- added link RL_EE, mass 0.001; collision sphere radius=0.01
- added link RR_EE, mass 0.001; collision sphere radius=0.01
Joints:
- removed joint FL_ee_joint
- removed joint FR_ee_joint
- removed joint RL_ee_joint
- removed joint RR_ee_joint
- added joint FL_EE_joint: type fixed, parent FL_calf, child FL_EE, origin xyz=0 0 -0.1 rpy=0 0 0
- added joint FR_EE_joint: type fixed, parent FR_calf, child FR_EE, origin xyz=0 0 -0.1 rpy=0 0 0
- added joint RL_EE_joint: type fixed, parent RL_calf, child RL_EE, origin xyz=0 0 -0.1 rpy=0 0 0
- added joint RR_EE_joint: type fixed, parent RR_calf, child RR_EE, origin xyz=0 0 -0.1 rpy=0 0 0
